File: SingleSystem1.brd (EAGLE design)
At the start: 170 x 110 mm, 7 parts, among them U2 SD_CARD_SOCKET, U3 XBEE

Commit message: done, now verifying
Parts:
- added 12+, GND: SE14, solpad:SE14
- added 3.3V, 5V, 9V: (no value), con-amp-quick:02P
- added 3DR: 653006114822, Wire_to_Board_Connectors_rev15d:653006114822
- added 5REG, 9REG: V_REG_317SMD, SparkFun-PowerIC:SOT223
- added A1_FTDI, A2_FTDI, GPS_FTDI, IMU_FTDI: (no value), con-amp-quick:06P
- added ANEMOMETER1, ANEMOMETER2: 61200622323, Wurth_Elektronik_Electromechanic_Wire_to_Board_Connectors_rev15c:61200622323
- added C1, C3: 1uF, SparkFun-Capacitors:0805
- added C13, C15: 0.1UF, SparkFun-Capacitors:0805
- added C14, C16: 1UF, SparkFun-Capacitors:0805
- added C2: 100uF, SparkFun-Capacitors:1206
- added C4: 10uF, SparkFun-Capacitors:0805
- added C5, C9: 0.022uF, SparkFun-Capacitors:0603-CAP
- added D2: (no value), Wuerth_Elektronik_LEDs_rev15b:1206
- added R13: 68.1k, resistor:M2012
- added R17: 100k, resistor:M2012
- added R2: (no value), resistor:M2012
- added R3: 750 ohms, adafruit:M2012
- added R4, R6: 240 ohms, adafruit:M2012
- added R5: 1.5k, adafruit:M2012
- added R7: 1.07k, resistor:M2012
- added R8: 5.62k, resistor:M2012
- added R9: 11.8k, resistor:M2012
- added U1: LMZ14203, SparkFun-PowerIC:TO-PMOD-7
- moved IMUCONNECTION 15.5 mm to (74.9, 15.2)
- moved U2 7.73 mm to (157.5, 15.2)
Connections:
- new net +12V: 12+.MP, 9REG.3, C1.1, C15.1, C4.1, D2.2, R13.2, R17.2, U1.1
- new net +9V: 5REG.3, 9REG.2, 9V.2, C13.1, C16.1, R6.2, U$1.VIN
- new net 3DR_RX: 3DR.3
- new net 3DR_TX: 3DR.2
- new net A1_PWR: ANEMOMETER1.2
- new net A2_PWR: ANEMOMETER2.2
- new net N$2: 5REG.1, R3.2, R4.1
- new net N$3: 9REG.1, R5.2, R6.1
- new net N$4: R13.1, R9.2, U1.3
- new net N$5: R17.1, U1.2
- new net N$6: C9.1, U1.5
- new net N$7: D2.1, R2.2
- new net N$8: C5.1, R7.2, R8.2, U1.6
- net +5V: now also 3DR.1, 5REG.2, 5V.2, C14.1, R4.2
- net 3.3V: now also 3.3V.2, C2.1, C3.1, C5.2, R8.1, U1.7
- net A1_IN_RX: now also ANEMOMETER1.5
- net A1_IN_TX: now also ANEMOMETER1.3
- net A1_RX: now also A1_FTDI.2
- net A1_TX: now also A1_FTDI.3
- net A2_IN_RX: now also ANEMOMETER2.5
- net A2_IN_TX: now also ANEMOMETER2.3
- net A2_RX: now also A2_FTDI.2
- net A2_TX: now also A2_FTDI.3
- net GND: now also 3.3V.1, 3DR.6, 5V.1, 9V.1, A1_FTDI.6, A2_FTDI.6, ANEMOMETER1.1, ANEMOMETER1.4, ANEMOMETER2.1, ANEMOMETER2.4, C1.2, C13.2, C14.2, C15.2, C16.2, C2.2, C3.2, C4.2, C9.2, GND.MP, GPS_FTDI.6, IMU_FTDI.6, R2.1, R3.1, R5.1, R7.1, R9.1, U$1.5V, U1.4, U1.EP
- net GPS_RX: now also GPS_FTDI.3, U$1.52
- net GPS_TX: now also GPS_FTDI.2, U$1.A11
- net IMU_RX: now also IMU_FTDI.3
- net IMU_TX: now also IMU_FTDI.2
Routing:
- net GND: track 0.00 -> 615.9 mm, vias 0 -> 2
- net 3.3V: track 0.00 -> 341.8 mm, vias 0 -> 8
- net GPS_RX: track 0.00 -> 231.9 mm, vias 0 -> 1
- net +9V: track 0.00 -> 229.7 mm, vias 0 -> 7
- net GPS_TX: track 0.00 -> 220.5 mm, vias 0 -> 3
- net +5V: track 0.00 -> 218.6 mm
- net A2_RX: track 0.00 -> 155.4 mm
- net A2_TX: track 0.00 -> 152.3 mm
- net IMU_TX: track 0.00 -> 151.9 mm, vias 0 -> 1
- net A1_RX: track 0.00 -> 151.9 mm
- net IMU_RX: track 0.00 -> 148.9 mm
- net A1_TX: track 0.00 -> 145.6 mm
- net A2_IN_RX: track 0.00 -> 144.9 mm
- net A1_IN_RX: track 0.00 -> 130.9 mm
- net +12V: track 0.00 -> 128.2 mm
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Other:
- outline, holes or cut-outs redrawn

Commit message: Done, Kanishke will verify
Parts:
- moved U3 17.8 mm to (49.5, 85.1), turned to 270 degrees
- moved U2 2.84 mm to (160.0, 16.5)
- flipped D2 to the top
Connections:
- net GND: now also U$1.GND_1; no longer U$1.5V
- net GPS_RX: now also U$1.A11; no longer U$1.52
- net GPS_TX: now also U$1.52; no longer U$1.A11
Routing:
- net GND: track 615.9 -> 671.0 mm, vias 2 -> 0
- net N$7: track 41.0 -> 71.7 mm, vias 2 -> 1
- net A1_RX: track 151.9 -> 179.7 mm
- net XBEE_RX: track 29.0 -> 53.3 mm
- net A1_TX: track 145.6 -> 169.1 mm
- net GPS_RX: track 231.9 -> 210.3 mm, vias 1 -> 3
- net XBEE_TX: track 19.9 -> 40.6 mm
- net 3.3V: track 341.8 -> 361.9 mm
- net A2_IN_RX: track 144.9 -> 128.1 mm, vias 0 -> 1
- net +5V: track 218.6 -> 207.9 mm
- net +12V: track 128.2 -> 138.9 mm, vias 0 -> 4
- net GPS_TX: track 220.5 -> 230.4 mm
- net A2_IN_TX: track 126.4 -> 120.7 mm, vias 2 -> 0
- net MISO: track 61.6 -> 57.1 mm, vias 0 -> 1
- net +9V: track 229.7 -> 233.2 mm, vias 7 -> 4
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Other:
- board text added: "FRONT"

Commit message: modified, verification is remaining
Parts:
- moved GND 12.7 mm to (101.6, 5.08)
- moved IMUCONNECTION 12.7 mm to (87.6, 15.2)
- moved 12+ 11.7 mm to (111.8, 5.08)
Routing:
- net N$7: track 71.7 -> 42.2 mm, vias 1 -> 3
- net IMU_RX: track 146.4 -> 171.7 mm, vias 1 -> 2
- net IMU_TX: track 150.3 -> 174.0 mm
- net +9V: track 233.2 -> 253.4 mm, vias 4 -> 5
- net 3.3V: track 361.9 -> 376.4 mm, vias 8 -> 7
- net +12V: track 138.9 -> 150.7 mm
- net +5V: track 207.9 -> 217.3 mm
- net GND: track 671.0 -> 675.0 mm
- net A2_IN_TX: track 120.7 -> 123.4 mm
- net GPS_RX: track 210.3 -> 212.7 mm
- net A1_RX: track 179.7 -> 177.5 mm
- net SCK: track 61.9 -> 60.5 mm
- net A2_IN_RX: track 128.1 -> 127.2 mm, vias 1 -> 2
- net A2_RX: track 155.4 -> 154.9 mm, vias 0 -> 1

Commit message: edited the pwr connections
Connections:
- removed net A1_PWR: ANEMOMETER1.2
- removed net A2_PWR: ANEMOMETER2.2
- removed net ANT_PWR: GPS(OEM615).20
- removed net GPS_PWR: GPS(OEM615).1
- net +12V: now also ANEMOMETER1.2, ANEMOMETER2.2
- net +9V: now also GPS(OEM615).20
- net 3.3V: now also GPS(OEM615).1
- net IMU_RX: now also IMUCONNECTION.7; no longer IMUCONNECTION.3
Routing:
- net +12V: track 150.7 -> 226.4 mm
- net GPS_TX: track 230.4 -> 275.3 mm, vias 3 -> 1
- net +9V: track 253.4 -> 219.6 mm, vias 5 -> 7
- net XBEE_TX: track 40.6 -> 74.2 mm
- net A2_TX: track 151.2 -> 179.0 mm
- net A1_IN_TX: track 121.6 -> 146.0 mm
- net 3.3V: track 376.4 -> 359.7 mm, vias 7 -> 8
- net GND: track 675.0 -> 659.4 mm, vias 0 -> 1
- net A1_RX: track 177.5 -> 167.4 mm, vias 0 -> 1
- net +5V: track 217.3 -> 225.0 mm
- net IMU_TX: track 174.0 -> 168.5 mm, vias 1 -> 2
- net GPS_RX: track 212.7 -> 207.7 mm
- net A2_RX: track 154.9 -> 159.2 mm
- net IMU_RX: track 171.7 -> 167.7 mm
- net A2_IN_TX: track 123.4 -> 120.9 mm
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Other:
- board text added: "SingleSystemV1.0 FDCL"

Commit message: edited 3DR
Connections:
- net 3DR_RX: now also U$1.TX0
- net 3DR_TX: now also U$1.RX0
Routing:
- net +9V: track 219.6 -> 312.8 mm, vias 7 -> 5
- net 3DR_RX: track 0.00 -> 86.7 mm
- net 3DR_TX: track 0.00 -> 86.6 mm
- net GPS_TX: track 275.3 -> 209.8 mm, vias 1 -> 4
- net XBEE_TX: track 74.2 -> 43.6 mm, vias 0 -> 2
- net A2_TX: track 179.0 -> 150.8 mm
- net GND: track 659.4 -> 685.0 mm, vias 1 -> 3
- net A1_IN_TX: track 146.0 -> 125.3 mm, vias 2 -> 0
- net +5V: track 225.0 -> 239.8 mm
- net IMU_RX: track 167.7 -> 181.4 mm, vias 2 -> 1
- net +12V: track 226.4 -> 238.3 mm, vias 4 -> 6
- net 3.3V: track 359.7 -> 370.1 mm, vias 8 -> 5
- net IMU_TX: track 168.5 -> 178.8 mm, vias 2 -> 0
- net A1_IN_RX: track 132.9 -> 142.3 mm, vias 0 -> 1
- net A2_IN_RX: track 127.2 -> 133.4 mm
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