File: Single System/SingleSystem1.sch (EAGLE design)
At the start: 43 parts, among them U1 LMZ14203, U2 SD_CARD_SOCKET, U3 XBEE

Commit message: final done
Connections:
- net XBEE_RX: now also U3.DOUT; no longer U3.DIN
- net XBEE_TX: now also U3.DIN; no longer U3.DOUT
Changed lines of the file:
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@@
 </segment>
 <segment>
-<wire x1="198.12" y1="43.18" x2="208.28" y2="43.18" width="0.1524" layer="91"/>
-<pinref part="U3" gate="G$1" pin="DOUT"/>
-<label x="198.12" y="43.18" size="1.778" layer="95" rot="R180" xref="yes"/>
+<wire x1="198.12" y1="40.64" x2="208.28" y2="40.64" width="0.1524" layer="91"/>
+<pinref part="U3" gate="G$1" pin="DIN"/>
+<label x="198.12" y="40.64" size="1.778" layer="95" rot="R180" xref="yes"/>
 </segment>
 </net>
@@
 </segment>
 <segment>
-<wire x1="198.12" y1="40.64" x2="208.28" y2="40.64" width="0.1524" layer="91"/>
-<pinref part="U3" gate="G$1" pin="DIN"/>
-<label x="198.12" y="40.64" size="1.778" layer="95" rot="R180" xref="yes"/>
+<wire x1="198.12" y1="43.18" x2="208.28" y2="43.18" width="0.1524" layer="91"/>
+<pinref part="U3" gate="G$1" pin="DOUT"/>
+<label x="198.12" y="43.18" size="1.778" layer="95" rot="R180" xref="yes"/>
 </segment>
 </net>
